File: supply.sch (KiCad schematic (older format))
At the start: 36 parts, among them J1 MJ-3536, J2 2, J3 3, J4 1, J5 GND, J6 Conn_01x01_Female, J7 Conn_01x01_Female, J8 Conn_01x01_Female, J9 Conn_01x01_Female, SW1 TE6-1A-DC-1-PB, U1 LM5157, U2 LM386N-4/NOPB

Commit message: Add files via upload
Parts:
- added C5: 100uF, Capacitor_THT:C_Disc_D3.8mm_W2.6mm_P2.50mm, symbol Device:C
- added C6: 0.1uF, Capacitor_THT:C_Disc_D3.8mm_W2.6mm_P2.50mm, symbol Device:C
- C11: value 10pF -> 220 µF; footprint Capacitor_THT:C_Disc_D3.8mm_W2.6mm_P2.50mm -> Capacitor_THT:CP_Radial_D6.3mm_P2.50mm
- D1: value BAT46 -> SB130-T
- R7: value 100 -> 10
Connections:
- net GND: now also C5.1, C6.1
- net at C10.2, C9.2, D1.1 (K)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: now also D2.2 (A), PTC1.2, C5.2, C6.2; no longer PTC1.1
- new net: PTC1.1, R3.1
Other:
- moved on the sheet: C10, C9, D1, D2, PTC1, R5, R6, R8
Changed lines of the file:
@@
 	4400 3800 3900 3800
-Wire Wire Line
-	4200 5650 6100 5650
 Wire Wire Line
 	6100 5650 6100 5150
@@
 L Device:D_Schottky D1
 U 1 1 60D4E839
-P 6850 4200
-F 0 "D1" H 6850 3983 50  0000 C CNN
-F 1 "BAT46" H 6850 4074 50  0000 C CNN
-F 2 "Diode_THT:D_DO-35_SOD27_P7.62mm_Horizontal" H 6850 4200 50  0001 C CNN
-F 3 "~" H 6850 4200 50  0001 C CNN
-	1    6850 4200
-	-1   0    0    1
-$EndComp
-Wire Wire Line
-	6700 4200 6100 4200
+P 6350 4200
+F 0 "D1" H 6350 3983 50  0000 C CNN
+F 1 "SB130-T" H 6350 4074 50  0000 C CNN
+F 2 "Diode_THT:D_DO-35_SOD27_P7.62mm_Horizontal" H 6350 4200 50  0001 C CNN
+F 3 "~" H 6350 4200 50  0001 C CNN
+	1    6350 4200
+	-1   0    0    1
+$EndComp
 $Comp
 L Device:R R5
 U 1 1 60D52774
-P 7250 4350
-F 0 "R5" H 7320 4396 50  0000 L CNN
-F 1 "118K" H 7320 4305 50  0000 L CNN
-F 2 "Resistor_THT:R_Axial_DIN0207_L6.3mm_D2.5mm_P7.62mm_Horizontal" V 7180 4350 50  0001 C CNN
-F 3 "~" H 7250 4350 50  0001 C CNN
-	1    7250 4350
+P 6800 4350
+F 0 "R5" H 6870 4396 50  0000 L CNN
+F 1 "118K" H 6870 4305 50  0000 L CNN
+F 2 "Resistor_THT:R_Axial_DIN0207_L6.3mm_D2.5mm_P7.62mm_Horizontal" V 6730 4350 50  0001 C CNN
+F 3 "~" H 6800 4350 50  0001 C CNN
+	1    6800 4350
 	1    0    0    -1
 $EndComp
@@
 L Device:R R6
 U 1 1 60D52C1F
-P 7250 4950
-F 0 "R6" H 7320 4996 50  0000 L CNN
-F 1 "2.49K" H 7320 4905 50  0000 L CNN
-F 2 "Resistor_THT:R_Axial_DIN0207_L6.3mm_D2.5mm_P7.62mm_Horizontal" V 7180 4950 50  0001 C CNN
-F 3 "~" H 7250 4950 50  0001 C CNN
-	1    7250 4950
-	1    0    0    -1
-$EndComp
-Wire Wire Line
-	7000 4200 7250 4200
-Wire Wire Line
-	7250 4500 7250 4650
-Wire Wire Line
-	7250 5100 7250 5650
-Wire Wire Line
-	7250 5650 6100 5650
+P 6800 4950
+F 0 "R6" H 6870 4996 50  0000 L CNN
+F 1 "2.49K" H 6870 4905 50  0000 L CNN
+F 2 "Resistor_THT:R_Axial_DIN0207_L6.3mm_D2.5mm_P7.62mm_Horizontal" V 6730 4950 50  0001 C CNN
+F 3 "~" H 6800 4950 50  0001 C CNN
+	1    6800 4950
+	1    0    0    -1
+$EndComp
+Wire Wire Line
+	6800 4500 6800 4650
+Wire Wire Line
+	6800 5100 6800 5650
+Wire Wire Line
+	6800 5650 6100 5650
 Connection ~ 6100 5650
-Wire Wire Line
-	5850 4650 7250 4650
-Connection ~ 7250 4650
-Wire Wire Line
-	7250 4650 7250 4800
+Connection ~ 6800 4650
+Wire Wire Line
+	6800 4650 6800 4800
 $Comp
 L Device:C C9
 U 1 1 60D5D442
-P 7850 4700
-F 0 "C9" H 7735 4654 50  0000 R CNN
-F 1 "1nF" H 7735 4745 50  0000 R CNN
-F 2 "Capacitor_THT:C_Disc_D3.8mm_W2.6mm_P2.50mm" H 7888 4550 50  0001 C CNN
-F 3 "~" H 7850 4700 50  0001 C CNN
-	1    7850 4700
+P 7400 4700
+F 0 "C9" H 7285 4654 50  0000 R CNN
+F 1 "1nF" H 7285 4745 50  0000 R CNN
+F 2 "Capacitor_THT:C_Disc_D3.8mm_W2.6mm_P2.50mm" H 7438 4550 50  0001 C CNN
+F 3 "~" H 7400 4700 50  0001 C CNN
+	1    7400 4700
 	-1   0    0    1
 $EndComp
@@
 L Device:C C10
 U 1 1 60D5E056
-P 8500 4700
-F 0 "C10" H 8385 4654 50  0000 R CNN
-F 1 "100nF" H 8385 4745 50  0000 R CNN
-F 2 "Capacitor_THT:C_Disc_D3.8mm_W2.6mm_P2.50mm" H 8538 4550 50  0001 C CNN
-F 3 "~" H 8500 4700 50  0001 C CNN
-	1    8500 4700
-	-1   0    0    1
-$EndComp
-Wire Wire Line
-	7250 4200 7850 4200
-Wire Wire Line
-	7850 4200 7850 4550
-Connection ~ 7250 4200
-Wire Wire Line
-	7850 4850 7850 5650
-Wire Wire Line
-	7850 5650 7250 5650
-Connection ~ 7250 5650
-Wire Wire Line
-	8500 4850 8500 5650
-Wire Wire Line
-	8500 5650 7850 5650
-Connection ~ 7850 5650
-Wire Wire Line
-	8500 4550 8500 4200
-Wire Wire Line
-	8500 4200 7850 4200
-Connection ~ 7850 4200
+P 8050 4700
+F 0 "C10" H 7935 4654 50  0000 R CNN
+F 1 "100nF" H 7935 4745 50  0000 R CNN
+F 2 "Capacitor_THT:C_Disc_D3.8mm_W2.6mm_P2.50mm" H 8088 4550 50  0001 C CNN
+F 3 "~" H 8050 4700 50  0001 C CNN
+	1    8050 4700
+	-1   0    0    1
+$EndComp
+Wire Wire Line
+	6800 4200 7400 4200
+Wire Wire Line
+	7400 4200 7400 4550
+Connection ~ 6800 4200
+Wire Wire Line
+	7400 4850 7400 5650
+Wire Wire Line
+	7400 5650 6800 5650
+Connection ~ 6800 5650
+Wire Wire Line
+	8050 4850 8050 5650
+Wire Wire Line
+	8050 5650 7400 5650
+Connection ~ 7400 5650
+Wire Wire Line
+	8050 4550 8050 4200
+Wire Wire Line
+	8050 4200 7400 4200
+Connection ~ 7400 4200
 Wire Wire Line
 	6250 3650 6250 3350
-Connection ~ 8500 4200
+Connection ~ 8050 4200
 $Comp
 L Switch:SW_SPST SW1
@@
 	2100 3800 1850 3800
 Wire Wire Line
-	8500 4200 8600 4200
-Wire Wire Line
-	9200 5650 8500 5650
-Connection ~ 8500 5650
+	8750 5650 8050 5650
+Connection ~ 8050 5650
 Wire Wire Line
 	3550 3150 3550 2950
@@
 L keyboard:PTC PTC1
 U 1 1 60D2EB90
-P 8850 4200
-F 0 "PTC1" H 8850 4515 50  0000 C CNN
-F 1 "YPEL6250T" H 8850 4424 50  0000 C CNN
-F 2 "Resistor_THT:R_Axial_DIN0204_L3.6mm_D1.6mm_P5.08mm_Horizontal" V 8850 4200 60  0001 C CNN
-F 3 "" V 8850 4200 60  0000 C CNN
-	1    8850 4200
-	1    0    0    -1
-$EndComp
-Wire Wire Line
-	9100 4200 9200 4200
+P 8300 3650
+F 0 "PTC1" H 8300 3965 50  0000 C CNN
+F 1 "YPEL6250T" H 8300 3874 50  0000 C CNN
+F 2 "Resistor_THT:R_Axial_DIN0204_L3.6mm_D1.6mm_P5.08mm_Horizontal" V 8300 3650 60  0001 C CNN
+F 3 "" V 8300 3650 60  0000 C CNN
+	1    8300 3650
+	1    0    0    -1
+$EndComp
 $Comp
 L Device:R R8
 U 1 1 60D30BFB
-P 9200 5450
-F 0 "R8" H 9270 5496 50  0000 L CNN
-F 1 "12K" H 9270 5405 50  0000 L CNN
-F 2 "Resistor_THT:R_Axial_DIN0204_L3.6mm_D1.6mm_P7.62mm_Horizontal" V 9130 5450 50  0001 C CNN
-F 3 "~" H 9200 5450 50  0001 C CNN
-	1    9200 5450
+P 8750 5450
+F 0 "R8" H 8820 5496 50  0000 L CNN
+F 1 "12K" H 8820 5405 50  0000 L CNN
+F 2 "Resistor_THT:R_Axial_DIN0204_L3.6mm_D1.6mm_P7.62mm_Horizontal" V 8680 5450 50  0001 C CNN
+F 3 "~" H 8750 5450 50  0001 C CNN
+	1    8750 5450
 	1    0    0    -1
 $EndComp
@@
 L Device:LED D2
 U 1 1 60D31DED
-P 9200 4700
-F 0 "D2" V 9239 4582 50  0000 R CNN
-F 1 "18-032.0055L" V 9148 4582 50  0000 R CNN
-F 2 "LED_THT:LED_D2.0mm_W4.8mm_H2.5mm_FlatTop" H 9200 4700 50  0001 C CNN
-F 3 "~" H 9200 4700 50  0001 C CNN
-	1    9200 4700
+P 8750 4700
+F 0 "D2" V 8789 4582 50  0000 R CNN
+F 1 "18-032.0055L" V 8698 4582 50  0000 R CNN
+F 2 "LED_THT:LED_D2.0mm_W4.8mm_H2.5mm_FlatTop" H 8750 4700 50  0001 C CNN
+F 3 "~" H 8750 4700 50  0001 C CNN
+	1    8750 4700
 	0    -1   -1   0
 $EndComp
 Wire Wire Line
-	9200 4200 9200 3650
-Wire Wire Line
-	6250 3650 9200 3650
-Connection ~ 9200 4200
-Wire Wire Line
-	9200 5600 9200 5650
-Wire Wire Line
-	9200 4200 9200 4550
-Wire Wire Line
-	9200 4850 9200 5300
+	8750 4200 8750 3650
+Connection ~ 8750 4200
+Wire Wire Line
+	8750 5600 8750 5650
+Wire Wire Line
+	8750 4200 8750 4550
+Wire Wire Line
+	8750 4850 8750 5300
 Wire Wire Line
 	1800 6250 1800 6450
@@
 P 3900 1850
 F 0 "R7" H 3970 1896 50  0000 L CNN
-F 1 "100" H 3970 1805 50  0000 L CNN
+F 1 "10" H 3970 1805 50  0000 L CNN
 F 2 "Resistor_THT:R_Axial_DIN0207_L6.3mm_D2.5mm_P7.62mm_Horizontal" V 3830 1850 50  0001 C CNN
 F 3 "~" H 3900 1850 50  0001 C CNN
@@
 P 4550 1050
 F 0 "C11" V 4298 1050 50  0000 C CNN
-F 1 "10pF" V 4389 1050 50  0000 C CNN
-F 2 "Capacitor_THT:C_Disc_D3.8mm_W2.6mm_P2.50mm" H 4588 900 50  0001 C CNN
+F 1 "220 µF" V 4389 1050 50  0000 C CNN
+F 2 "Capacitor_THT:CP_Radial_D6.3mm_P2.50mm" H 4588 900 50  0001 C CNN
 F 3 "~" H 4550 1050 50  0001 C CNN
 	1    4550 1050
@@
 Text Label 4950 2700 0    50   ~ 0
 5
+$Comp
+L Device:C C5
+U 1 1 60D4F7C0
+P 9600 4750
+F 0 "C5" H 9485 4704 50  0000 R CNN
+F 1 "100uF" H 9485 4795 50  0000 R CNN
+F 2 "Capacitor_THT:C_Disc_D3.8mm_W2.6mm_P2.50mm" H 9638 4600 50  0001 C CNN
+F 3 "~" H 9600 4750 50  0001 C CNN
+	1    9600 4750
+	-1   0    0    1
+$EndComp
+Wire Wire Line
+	9600 4200 8750 4200
+Wire Wire Line
+	9600 4200 9600 4600
+Wire Wire Line
+	9600 4900 9600 5650
+Wire Wire Line
+	9600 5650 8750 5650
+Connection ~ 8750 5650
+$Comp
+L Device:C C6
+U 1 1 60D627B5
+P 10200 4750
+F 0 "C6" H 10085 4704 50  0000 R CNN
+F 1 "0.1uF" H 10085 4795 50  0000 R CNN
+F 2 "Capacitor_THT:C_Disc_D3.8mm_W2.6mm_P2.50mm" H 10238 4600 50  0001 C CNN
+F 3 "~" H 10200 4750 50  0001 C CNN
+	1    10200 4750
+	-1   0    0    1
+$EndComp
+Wire Wire Line
+	9600 4200 10200 4200
+Connection ~ 9600 4200
+Wire Wire Line
+	10200 4900 10200 5650
+Wire Wire Line
+	10200 5650 9600 5650
+Connection ~ 9600 5650
+Wire Wire Line
+	10200 4600 10200 4200
+Wire Wire Line
+	6200 4200 6100 4200
+Wire Wire Line
+	5850 4650 6800 4650
+Wire Wire Line
+	6250 3650 8050 3650
+Wire Wire Line
+	4200 5650 6100 5650
+Wire Wire Line
+	6500 4200 6800 4200
+Wire Wire Line
+	8550 3650 8750 3650
+Wire Wire Line
+	8050 4200 8750 4200
 $EndSCHEMATC

Commit message: Add files via upload
Parts:
- removed C5: 100uF, Capacitor_THT:C_Disc_D3.8mm_W2.6mm_P2.50mm, symbol Device:C
- added C5: 100uF, Capacitor_THT:CP_Radial_D8.0mm_P3.50mm, symbol Device:CP
Connections:
- net GND: now also C5.2
- net at C10.2, C6.2, C9.2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: now also C5.1
Changed lines of the file:
@@
 Text Label 4950 2700 0    50   ~ 0
 5
-$Comp
-L Device:C C5
-U 1 1 60D4F7C0
-P 9600 4750
-F 0 "C5" H 9485 4704 50  0000 R CNN
-F 1 "100uF" H 9485 4795 50  0000 R CNN
-F 2 "Capacitor_THT:C_Disc_D3.8mm_W2.6mm_P2.50mm" H 9638 4600 50  0001 C CNN
-F 3 "~" H 9600 4750 50  0001 C CNN
-	1    9600 4750
-	-1   0    0    1
-$EndComp
-Wire Wire Line
-	9600 4200 8750 4200
-Wire Wire Line
-	9600 4200 9600 4600
-Wire Wire Line
-	9600 4900 9600 5650
-Wire Wire Line
-	9600 5650 8750 5650
 Connection ~ 8750 5650
-$Comp
-L Device:C C6
-U 1 1 60D627B5
-P 10200 4750
-F 0 "C6" H 10085 4704 50  0000 R CNN
-F 1 "0.1uF" H 10085 4795 50  0000 R CNN
-F 2 "Capacitor_THT:C_Disc_D3.8mm_W2.6mm_P2.50mm" H 10238 4600 50  0001 C CNN
-F 3 "~" H 10200 4750 50  0001 C CNN
-	1    10200 4750
-	-1   0    0    1
-$EndComp
-Wire Wire Line
-	9600 4200 10200 4200
-Connection ~ 9600 4200
 Wire Wire Line
 	10200 4900 10200 5650
-Wire Wire Line
-	10200 5650 9600 5650
-Connection ~ 9600 5650
 Wire Wire Line
 	10200 4600 10200 4200
@@
 Wire Wire Line
 	8050 4200 8750 4200
+$Comp
+L Device:C C6
+U 1 1 60D627B5
+P 10200 4750
+F 0 "C6" H 10085 4704 50  0000 R CNN
+F 1 "0.1uF" H 10085 4795 50  0000 R CNN
+F 2 "Capacitor_THT:C_Disc_D3.8mm_W2.6mm_P2.50mm" H 10238 4600 50  0001 C CNN
+F 3 "~" H 10200 4750 50  0001 C CNN
+	1    10200 4750
+	-1   0    0    1
+$EndComp
+Wire Wire Line
+	10200 5650 9600 5650
+Wire Wire Line
+	9600 5650 8750 5650
+Connection ~ 9600 5650
+Wire Wire Line
+	9600 4900 9600 5650
+Wire Wire Line
+	9600 4200 10200 4200
+Wire Wire Line
+	9600 4200 8750 4200
+Connection ~ 9600 4200
+Wire Wire Line
+	9600 4200 9600 4600
+$Comp
+L Device:CP C5
+U 1 1 60D58BED
+P 9600 4750
+F 0 "C5" H 9718 4796 50  0000 L CNN
+F 1 "100uF" H 9718 4705 50  0000 L CNN
+F 2 "Capacitor_THT:CP_Radial_D8.0mm_P3.50mm" H 9638 4600 50  0001 C CNN
+F 3 "~" H 9600 4750 50  0001 C CNN
+	1    9600 4750
+	1    0    0    -1
+$EndComp
 $EndSCHEMATC
